File: cart.kicad_sch (KiCad schematic)
At the start: 1 part, among them J4 CARTRIDGE EDGE

Commit message: board layout
Changed lines of the file:
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@@
 	)
 	(global_label "ESND"
-		(shape input)
+		(shape output)
 		(at 147.32 88.9 0)
 		(fields_autoplaced yes)
