File: DragonATXProto.kicad_pcb (KiCad board)
At the start: 2 copper layers, 169.6 x 229.8 mm, 28 parts, among them J1 PWR_SWITCH, J2 PWR_LED, J3 RESET, J4 CARTRIDGE EDGE, U1 TSN 1-2450

Commit message: board layout
Parts:
- added C4: 0.1uF, Capacitor_THT:C_Disc_D4.3mm_W1.9mm_P5.00mm, F.Cu at (69.0, 97.8)
- added C5: 22nF, Capacitor_THT:C_Disc_D5.0mm_W2.5mm_P5.00mm, F.Cu at (51.2, 71.4)
- added C6: 22nF, Capacitor_THT:C_Disc_D5.0mm_W2.5mm_P5.00mm, F.Cu at (56.3, 116.4)
- added C7: 22nF, Capacitor_THT:C_Disc_D5.0mm_W2.5mm_P5.00mm, F.Cu at (59.2, 71.4)
- added C8: 22nF, Capacitor_THT:C_Disc_D5.0mm_W2.5mm_P5.00mm, F.Cu at (59.1, 116.4)
- added C9: 0.01uF, Capacitor_THT:C_Disc_D4.3mm_W1.9mm_P5.00mm, F.Cu at (56.3, 57.4)
- added D4: 1N914, Diode_THT:D_DO-35_SOD27_P12.70mm_Horizontal, F.Cu at (51.5, 78.7)
- added D5: 1N914, Diode_THT:D_DO-35_SOD27_P12.70mm_Horizontal, F.Cu at (51.5, 93.8)
- added D6: 1N914, Diode_THT:D_DO-35_SOD27_P12.70mm_Horizontal, F.Cu at (51.5, 90.8)
- added J5: Joystick ports, Connector_PinHeader_2.54mm:PinHeader_2x04_P2.54mm_Vertical, F.Cu at (76.7, 106.9)
- added J6: MD-40SM, Library:CUI_MD-40SM, F.Cu at (35.8, 124.4)
- added JP1: Jumper_2_Open, Jumper:SolderJumper-2_P1.3mm_Open_RoundedPad1.0x1.5mm, B.Cu at (77.6, 245.5)
- added JP2: Jumper_2_Open, Jumper:SolderJumper-2_P1.3mm_Open_RoundedPad1.0x1.5mm, B.Cu at (80.1, 242.2)
- added JP3: Jumper_2_Open, Jumper:SolderJumper-2_P1.3mm_Open_RoundedPad1.0x1.5mm, B.Cu at (82.6, 238.8)
- added L1: 3.3uH, Inductor_THT:L_Axial_L7.0mm_D3.3mm_P12.70mm_Horizontal_Fastron_MICC, F.Cu at (51.4, 61.2)
- added L2: 3.3uH, Inductor_THT:L_Axial_L7.0mm_D3.3mm_P12.70mm_Horizontal_Fastron_MICC, F.Cu at (64.1, 112.6)
- added L3: 3.3uH, Inductor_THT:L_Axial_L7.0mm_D3.3mm_P12.70mm_Horizontal_Fastron_MICC, F.Cu at (64.1, 108.6)
- added L4: 3.3uH, Inductor_THT:L_Axial_L7.0mm_D3.3mm_P12.70mm_Horizontal_Fastron_MICC, F.Cu at (51.4, 66.2)
- added PL11: DIN-6 J/S L, Library:DIN-6_DELTRON_671-0601_Horizontal, F.Cu at (43.3, 73.7)
- added PL12: DIN-6 J/S R, Library:DIN-6_DELTRON_671-0601_Horizontal, F.Cu at (43.3, 113.7)
- added R5: 4K7, Resistor_THT:R_Axial_DIN0204_L3.6mm_D1.6mm_P2.54mm_Vertical, F.Cu at (71.8, 95.0)
- added R6: 100R, Resistor_THT:R_Axial_DIN0204_L3.6mm_D1.6mm_P2.54mm_Vertical, F.Cu at (69.3, 95.0)
- added RL1: OMRON G2E, Library:OMRON_G2E, F.Cu at (57.8, 101.4)
- added TR1: BC141, Package_TO_SOT_THT:TO-92, F.Cu at (69.1, 89.5)
- added U2: ~, Library:QMTECH_XC7A15T, F.Cu at (117.7, 69.0)
- added Y1: CXO_DIP14, Oscillator:Oscillator_DIP-14, F.Cu at (158.8, 48.3)
- C1: footprint Capacitor_SMD:CP_Elec_6.3x5.4_Nichicon -> Capacitor_THT:CP_Radial_D8.0mm_P5.00mm
- C2: footprint Capacitor_SMD:C_0805_2012Metric_Pad1.18x1.45mm_HandSolder -> Capacitor_THT:C_Disc_D4.3mm_W1.9mm_P5.00mm
- C3: footprint Capacitor_SMD:CP_Elec_4x4.5 -> Capacitor_THT:CP_Radial_D8.0mm_P5.00mm
- D1, D2, D3: footprint Diode_SMD:D_SOD-323_HandSoldering -> Diode_THT:D_DO-34_SOD68_P7.62mm_Horizontal
- R1, R2, R3, R4: footprint Resistor_SMD:R_0805_2012Metric_Pad1.20x1.40mm_HandSolder -> Resistor_THT:R_Axial_DIN0204_L3.6mm_D1.6mm_P2.54mm_Vertical
- moved C2 136.4 mm to (191.1, 246.4), turned to 90 degrees
- moved R4 15.2 mm to (179.3, 98.7), turned to -90 degrees
- moved PL8 13.8 mm to (43.3, 93.7)
- moved R3 12.0 mm to (176.9, 108.6), turned to -90 degrees
- moved D1 7.66 mm to (181.9, 108.8), turned to 90 degrees
- moved R1 7.37 mm to (198.2, 244.6)
- moved J3 7.21 mm to (191.0, 251.2)
- moved J1 7.21 mm to (198.2, 251.2)
- moved D2 7.05 mm to (181.9, 111.1)
- moved D3 4.06 mm to (179.3, 103.5), turned to -90 degrees
- moved C1 2.30 mm to (191.1, 32.5)
- moved C3 1.94 mm to (185.0, 101.2)
- moved R2 0.99 mm to (194.6, 247.1)
Connections:
- F3 pad 2: +3V3 -> +3.3V
- PL1 pad a2: Luma -> Chroma
- PL1 pad a3: GND -> AD1
- PL1 pad a38: unconnected-(PL1A-Pin_a38-Pada38) -> VCLK
- PL1 pad b10: unconnected-(PL1A-Pin_b10-Padb10) -> ESND
- PL1 pad b2: Chroma -> Luma
- PL1 pad b3: AD1 -> GND
- PL2 pad a2: Luma -> Chroma
- PL2 pad a3: GND -> AD1
- PL2 pad a38: unconnected-(PL2A-Pin_a38-Pada38) -> VCLK
- PL2 pad b10: unconnected-(PL2A-Pin_b10-Padb10) -> ESND
- PL2 pad b2: Chroma -> Luma
- PL2 pad b3: AD1 -> GND
- PL3 pad a2: Luma -> Chroma
- PL3 pad a3: GND -> AD1
- PL3 pad a38: unconnected-(PL3A-Pin_a38-Pada38) -> VCLK
- PL3 pad b10: unconnected-(PL3A-Pin_b10-Padb10) -> ESND
- PL3 pad b2: Chroma -> Luma
- PL3 pad b3: AD1 -> GND
- PL4 pad a2: Luma -> Chroma
- PL4 pad a3: GND -> AD1
- PL4 pad a38: unconnected-(PL4A-Pin_a38-Pada38) -> VCLK
- PL4 pad b10: unconnected-(PL4A-Pin_b10-Padb10) -> ESND
- PL4 pad b2: Chroma -> Luma
- PL4 pad b3: AD1 -> GND
- PL6 pad a1: (no net) -> Composite
- PL6 pad a10: (no net) -> DL6
- PL6 pad a11: (no net) -> DL7
- PL6 pad a12: (no net) -> BS
- PL6 pad a13: (no net) -> BA
- PL6 pad a14: (no net) -> LIC
- PL6 pad a15: (no net) -> TSC
- PL6 pad a16: (no net) -> AVMA
- PL6 pad a17: (no net) -> CPU_BUSY
- PL6 pad a18: (no net) -> CART
- PL6 pad a19: (no net) -> EAR
- PL6 pad a2: (no net) -> Chroma
- PL6 pad a20: (no net) -> MIC
- PL6 pad a21: (no net) -> MOTOR
- PL6 pad a22: (no net) -> S0
- PL6 pad a23: (no net) -> S1
- PL6 pad a24: (no net) -> S2
- PL6 pad a25: (no net) -> S3
- PL6 pad a26: (no net) -> S4
- PL6 pad a27: (no net) -> P0
- PL6 pad a28: (no net) -> P1
- PL6 pad a29: (no net) -> P2
- PL6 pad a3: (no net) -> AD1
- PL6 pad a30: (no net) -> R0
- PL6 pad a31: (no net) -> R1
- PL6 pad a32: (no net) -> R2
- PL6 pad a33: (no net) -> CSS
- PL6 pad a34: (no net) -> ~{A}/G
- PL6 pad a35: (no net) -> GM0
- PL6 pad a36: (no net) -> GM1
- PL6 pad a37: (no net) -> GM2
- PL6 pad a38: (no net) -> VCLK
- PL6 pad a39: (no net) -> ~{HALT}
- PL6 pad a4: (no net) -> DL0
- PL6 pad a40: (no net) -> Q
- PL6 pad a41: (no net) -> E
- PL6 pad a42: (no net) -> A0
- PL6 pad a43: (no net) -> A1
- PL6 pad a5: (no net) -> DL1
- PL6 pad a6: (no net) -> DL2
- PL6 pad a7: (no net) -> DL3
- PL6 pad a8: (no net) -> DL4
- PL6 pad a9: (no net) -> DL5
- PL6 pad b1: (no net) -> +12V
- PL6 pad b10: (no net) -> ESND
- PL6 pad b11: (no net) -> EXTMEN
- PL6 pad b12: (no net) -> -5V
- PL6 pad b13: (no net) -> ~{NMI}p
- PL6 pad b14: (no net) -> ~{FIRQ}p
- PL6 pad b15: (no net) -> ~{IRQ}p
- PL6 pad b16: (no net) -> -12V
- PL6 pad b17: (no net) -> ~{NMI}
- PL6 pad b18: (no net) -> ~{FIRQ}
- PL6 pad b19: (no net) -> ~{IRQ}
- PL6 pad b2: (no net) -> Luma
- PL6 pad b20: (no net) -> ~{RESET}
- PL6 pad b21: (no net) -> Z0
- PL6 pad b22: (no net) -> Z1
- PL6 pad b23: (no net) -> Z2
- PL6 pad b24: (no net) -> Z3
- PL6 pad b25: (no net) -> Z4
- PL6 pad b26: (no net) -> Z5
- PL6 pad b27: (no net) -> Z6
- PL6 pad b28: (no net) -> Z7
- PL6 pad b29: (no net) -> Z8
- PL6 pad b3: (no net) -> GND
- PL6 pad b30: (no net) -> Z9
- PL6 pad b31: (no net) -> Z10
- PL6 pad b32: (no net) -> Z11
- PL6 pad b33: (no net) -> Z12
- PL6 pad b34: (no net) -> Z13
- PL6 pad b35: (no net) -> Z14
- PL6 pad b36: (no net) -> Z15
- PL6 pad b37: (no net) -> Z16
- PL6 pad b38: (no net) -> Z17
- PL6 pad b39: (no net) -> Z18
- PL6 pad b4: (no net) -> AD2
- PL6 pad b40: (no net) -> Z19
- PL6 pad b41: (no net) -> Z20
- PL6 pad b42: (no net) -> Z21
- PL6 pad b43: (no net) -> +5V
- PL6 pad b5: (no net) -> AUDIO_L
- PL6 pad b6: (no net) -> AUDIO_M
- PL6 pad b7: (no net) -> AUDIO_R
- PL6 pad b8: (no net) -> +3.3V
- PL6 pad b9: (no net) -> R/~{W}
- PL7 pad a2: Luma -> Chroma
- PL7 pad a3: GND -> AD1
- PL7 pad a38: unconnected-(PL7A-Pin_a38-Pada38) -> VCLK
- PL7 pad b10: unconnected-(PL7A-Pin_b10-Padb10) -> ESND
- PL7 pad b2: Chroma -> Luma
- PL7 pad b3: AD1 -> GND
Routing:
- net +5V: track 0.00 -> 588.0 mm, vias 0 -> 9
- net +12V: track 0.00 -> 547.8 mm, vias 0 -> 3
- net -5V: track 0.00 -> 368.2 mm, vias 0 -> 2
- net VCLK: track 0.00 -> 300.6 mm, vias 0 -> 1
- net R/~{W}: track 0.00 -> 293.5 mm, vias 0 -> 1
- net P2: track 0.00 -> 292.2 mm, vias 0 -> 1
- net R2: track 0.00 -> 270.3 mm, vias 0 -> 1
- net +3.3V: track 0.00 -> 259.7 mm, vias 0 -> 2
- net ~{NMI}p: track 0.00 -> 254.4 mm, vias 0 -> 3
- net EXTMEN: track 0.00 -> 249.6 mm, vias 0 -> 1
- net ESND: track 0.00 -> 246.2 mm, vias 0 -> 1
- net R1: track 0.00 -> 240.7 mm
- net Z11: track 0.00 -> 240.3 mm
- net DL0: track 0.00 -> 236.5 mm
- net A15: track 0.00 -> 234.4 mm
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Other:
- board text added: "CART"
- board text added: "PWR LED"
- board text added: "PWR SW"
- board text added: "RST"

Commit message: add notes
Parts:
- added C10: 0.1uF, Capacitor_SMD:C_0603_1608Metric, F.Cu at (97.4, 105.6)
- added C11: 0.1uF, Capacitor_SMD:C_0603_1608Metric, F.Cu at (104.8, 105.5)
- added C12: 0.1uF, Capacitor_SMD:C_0603_1608Metric, F.Cu at (133.6, 105.7)
- added C13: 0.1uF, Capacitor_SMD:C_0603_1608Metric, F.Cu at (141.7, 106.2)
- added C14: 0.1uF, Capacitor_SMD:C_0603_1608Metric, F.Cu at (157.2, 107.6)
- added C15: 0.1uF, Capacitor_SMD:C_0603_1608Metric, F.Cu at (97.4, 101.8)
- added C16: 0.1uF, Capacitor_SMD:C_0603_1608Metric, F.Cu at (104.8, 101.6)
- added C17: 0.1uF, Capacitor_SMD:C_0603_1608Metric, F.Cu at (133.6, 101.6)
- added C18: 0.1uF, Capacitor_SMD:C_0603_1608Metric, F.Cu at (142.4, 102.5)
- added C19: 0.1uF, Capacitor_SMD:C_0603_1608Metric, F.Cu at (157.2, 101.7)
- added C20: 0.1uF, Capacitor_SMD:C_0603_1608Metric, F.Cu at (133.9, 47.5)
- added C21: 0.1uF, Capacitor_SMD:C_0603_1608Metric, F.Cu at (126.4, 47.4)
- added R10: 220R, Resistor_SMD:R_0603_1608Metric, F.Cu at (87.5, 51.2)
- added R11: 220R, Resistor_SMD:R_0603_1608Metric, F.Cu at (87.5, 48.6)
- added R12: 220R, Resistor_SMD:R_0603_1608Metric, F.Cu at (87.5, 46.1)
- added R13: 220R, Resistor_SMD:R_0603_1608Metric, F.Cu at (87.5, 43.6)
- added R14: 220R, Resistor_SMD:R_0603_1608Metric, F.Cu at (87.4, 58.8)
- added R15: 220R, Resistor_SMD:R_0603_1608Metric, F.Cu at (87.4, 61.3)
- added R16: 220R, Resistor_SMD:R_0603_1608Metric, F.Cu at (87.4, 63.9)
- added R17: 220R, Resistor_SMD:R_0603_1608Metric, F.Cu at (147.8, 84.2)
- added R18: 220R, Resistor_SMD:R_0603_1608Metric, F.Cu at (147.8, 81.7)
- added R19: 220R, Resistor_SMD:R_0603_1608Metric, F.Cu at (147.8, 79.2)
- added R20: 220R, Resistor_SMD:R_0603_1608Metric, F.Cu at (147.8, 76.6)
- added R21: 220R, Resistor_SMD:R_0603_1608Metric, F.Cu at (147.8, 74.0)
- added R22: 220R, Resistor_SMD:R_0603_1608Metric, F.Cu at (147.8, 71.5)
- added R23: 220R, Resistor_SMD:R_0603_1608Metric, F.Cu at (147.8, 69.0)
- added R24: 220R, Resistor_SMD:R_0603_1608Metric, F.Cu at (147.8, 66.4)
- added R25: 220R, Resistor_SMD:R_0603_1608Metric, F.Cu at (147.8, 63.9)
- added R26: 220R, Resistor_SMD:R_0603_1608Metric, F.Cu at (147.8, 61.3)
- added R27: 220R, Resistor_SMD:R_0603_1608Metric, F.Cu at (147.8, 58.8)
- added R28: 220R, Resistor_SMD:R_0603_1608Metric, F.Cu at (147.8, 56.3)
- added R29: 220R, Resistor_SMD:R_0603_1608Metric, F.Cu at (147.8, 53.7)
- added R30: 220R, Resistor_SMD:R_0603_1608Metric, F.Cu at (160.0, 56.7)
- added R31: 220R, Resistor_SMD:R_0603_1608Metric, F.Cu at (161.7, 56.7)
- added R32: 220R, Resistor_SMD:R_0603_1608Metric, F.Cu at (163.3, 56.7)
- added R33: 220R, Resistor_SMD:R_0603_1608Metric, F.Cu at (138.3, 56.2)
- added R34: 220R, Resistor_SMD:R_0603_1608Metric, F.Cu at (87.5, 41.0)
- added R7: 220R, Resistor_SMD:R_0603_1608Metric, F.Cu at (87.5, 66.4)
- added R8: 220R, Resistor_SMD:R_0603_1608Metric, F.Cu at (87.5, 56.3)
- added R9: 220R, Resistor_SMD:R_0603_1608Metric, F.Cu at (87.5, 53.7)
- added U3: TXU0104PWR, Library:TSSOP_0104PWR, F.Cu at (129.8, 106.9)
- added U4: TXU0104PWR, Library:TSSOP_0104PWR, F.Cu at (93.7, 106.9)
- added U5: TXB0104PWR, Library:TSSOP_0104PWR, F.Cu at (137.3, 106.9)
- added U6: TXB0104PWR, Library:TSSOP_0104PWR, F.Cu at (153.3, 107.0)
- added U7: TXU0104PWR, Library:TSSOP_0104PWR, F.Cu at (101.2, 106.9)
- added U8: TXB0104PWR, Library:TSSOP_0104PWR, F.Cu at (130.1, 51.3)
Connections:
- U2 pad 10: unconnected-(U2A-R7-Pad10) -> DL5
- U2 pad 11: unconnected-(U2A-R6-Pad11) -> Net-(U2A-R6)
- U2 pad 12: unconnected-(U2A-T5-Pad12) -> DL4
- U2 pad 13: unconnected-(U2A-R5-Pad13) -> Net-(U2A-R5)
- U2 pad 14: unconnected-(U2A-T4-Pad14) -> DL3
- U2 pad 15: unconnected-(U2A-U6-Pad15) -> Z0
- U2 pad 16: unconnected-(U2A-U5-Pad16) -> DL2
- U2 pad 17: unconnected-(U2A-V4-Pad17) -> Z1
- U2 pad 18: unconnected-(U2A-U4-Pad18) -> DL1
- U2 pad 19: unconnected-(U2A-V3-Pad19) -> Z2
- U2 pad 20: unconnected-(U2A-V2-Pad20) -> DL0
- U2 pad 21: unconnected-(U2A-U2-Pad21) -> Z3
- U2 pad 22: unconnected-(U2A-U1-Pad22) -> Net-(U2A-U1)
- U2 pad 23: unconnected-(U2A-P4-Pad23) -> Z4
- U2 pad 24: unconnected-(U2A-T3-Pad24) -> Net-(U2A-T3)
- U2 pad 25: unconnected-(U2A-R3-Pad25) -> Z5
- U2 pad 26: unconnected-(U2A-T2-Pad26) -> Net-(U2A-T2)
- U2 pad 27: unconnected-(U2A-N4-Pad27) -> Z6
- U2 pad 28: unconnected-(U2A-P3-Pad28) -> Net-(U2A-P3)
- U2 pad 29: unconnected-(U2A-M6-Pad29) -> Z7
- U2 pad 30: unconnected-(U2A-M5-Pad30) -> Net-(U2A-M5)
- U2 pad 31: unconnected-(U2A-L5-Pad31) -> Z8
- U2 pad 32: unconnected-(U2A-L4-Pad32) -> Net-(U2A-L4)
- U2 pad 33: unconnected-(U2A-K3-Pad33) -> Z9
- U2 pad 34: unconnected-(U2A-K5-Pad34) -> Net-(U2A-K5)
- U2 pad 35: unconnected-(U2A-P1-Pad35) -> Z10
- U2 pad 36: unconnected-(U2A-R1-Pad36) -> Net-(U2A-R1)
- U2 pad 37: unconnected-(U2A-N1-Pad37) -> Z11
- U2 pad 38: unconnected-(U2A-N2-Pad38) -> Net-(U2A-N2)
- U2 pad 39: unconnected-(U2A-M2-Pad39) -> Z12
- U2 pad 40: unconnected-(U2A-M1-Pad40) -> Net-(U2A-M1)
- U2 pad 41: unconnected-(U2A-J5-Pad41) -> Z13
- U2 pad 42: unconnected-(U2A-J4-Pad42) -> Net-(U2A-J4)
- U2 pad 43: unconnected-(U2A-J6-Pad43) -> Z14
- U2 pad 44: unconnected-(U2A-K6-Pad44) -> Net-(U2A-K6)
- U2 pad 45: unconnected-(U2A-L2-Pad45) -> Z15
- U2 pad 46: unconnected-(U2A-L3-Pad46) -> Net-(U2A-L3)
- U2 pad 47: unconnected-(U2A-K2-Pad47) -> Z16
- U2 pad 48: unconnected-(U2A-K1-Pad48) -> Net-(U2A-K1)
- U2 pad 5: unconnected-(U2A-V8-Pad5) -> Net-(U2A-V8)
- U2 pad 55: unconnected-(U2B-F18-Pad55) -> Net-(U2B-F18)
- U2 pad 56: unconnected-(U2B-G17-Pad56) -> Net-(U2B-G17)
- U2 pad 57: unconnected-(U2B-E18-Pad57) -> Net-(U2B-E18)
- U2 pad 58: unconnected-(U2B-F17-Pad58) -> Net-(U2B-F17)
- U2 pad 59: unconnected-(U2B-D18-Pad59) -> Net-(U2B-D18)
- U2 pad 6: unconnected-(U2A-V7-Pad6) -> DL7
- U2 pad 60: unconnected-(U2B-E17-Pad60) -> Net-(U2B-E17)
- U2 pad 61: unconnected-(U2B-C17-Pad61) -> Net-(U2B-C17)
- U2 pad 62: unconnected-(U2B-C18-Pad62) -> Net-(U2B-C18)
- U2 pad 63: unconnected-(U2B-G15-Pad63) -> Net-(U2B-G15)
- U2 pad 65: unconnected-(U2B-F15-Pad65) -> Net-(U2B-F15)
- U2 pad 67: unconnected-(U2B-E16-Pad67) -> Net-(U2B-E16)
- U2 pad 68: unconnected-(U2B-E15-Pad68) -> Net-(U2B-E15)
- U2 pad 69: unconnected-(U2B-D16-Pad69) -> Net-(U2B-D16)
- U2 pad 7: unconnected-(U2A-U7-Pad7) -> Net-(U2A-U7)
- U2 pad 70: unconnected-(U2B-D15-Pad70) -> Net-(U2B-D15)
- U2 pad 71: unconnected-(U2B-A17-Pad71) -> Net-(U2B-A17)
- U2 pad 72: unconnected-(U2B-B17-Pad72) -> Net-(U2B-B17)
- U2 pad 73: unconnected-(U2B-C16-Pad73) -> Net-(U2B-C16)
- U2 pad 74: unconnected-(U2B-B16-Pad74) -> Net-(U2B-B16)
- U2 pad 75: unconnected-(U2B-A15-Pad75) -> Net-(U2B-A15)
- U2 pad 76: unconnected-(U2B-B15-Pad76) -> Z21
- U2 pad 77: unconnected-(U2B-A14-Pad77) -> Net-(U2B-A14)
- U2 pad 78: unconnected-(U2B-B14-Pad78) -> Z20
- U2 pad 79: unconnected-(U2B-C14-Pad79) -> Net-(U2B-C14)
- U2 pad 8: unconnected-(U2A-V6-Pad8) -> DL6
- U2 pad 80: unconnected-(U2B-D14-Pad80) -> Z19
- U2 pad 81: unconnected-(U2B-C13-Pad81) -> Net-(U2B-C13)
- U2 pad 82: unconnected-(U2B-D13-Pad82) -> Z18
- U2 pad 83: unconnected-(U2B-A13-Pad83) -> Net-(U2B-A13)
- U2 pad 84: unconnected-(U2B-C12-Pad84) -> Z17
- U2 pad 85: unconnected-(U2B-F14-Pad85) -> Net-(U2B-F14)
- U2 pad 86: unconnected-(U2B-E13-Pad86) -> Net-(U2B-E13)
- U2 pad 87: unconnected-(U2B-B12-Pad87) -> Net-(U2B-B12)
- U2 pad 88: unconnected-(U2B-A12-Pad88) -> Net-(U2B-A12)
- U2 pad 89: unconnected-(U2B-C11-Pad89) -> Net-(U2B-C11)
- U2 pad 9: unconnected-(U2A-T7-Pad9) -> Net-(U2A-T7)
- U2 pad 90: unconnected-(U2B-B11-Pad90) -> Net-(U2B-B11)
- U2 pad 91: unconnected-(U2B-D11-Pad91) -> Net-(U2B-D11)
- U2 pad 93: unconnected-(U2B-C9-Pad93) -> Net-(U2B-C9)
- Y1 pad 1: +5V -> +3.3V
- Y1 pad 14: +5V -> +3.3V
Routing:
- net +3.3V: track 259.7 -> 410.0 mm, vias 2 -> 7
- net P1: track 218.9 -> 105.3 mm
- net P0: track 211.8 -> 105.3 mm
- net +5V: track 588.0 -> 675.9 mm, vias 9 -> 22
- net EXTMEN: track 249.6 -> 327.9 mm, vias 1 -> 2
- net P2: track 292.2 -> 215.5 mm
- net R2: track 270.3 -> 205.0 mm
- net S4: track 204.4 -> 155.5 mm, vias 0 -> 2
- net VCLK: track 300.6 -> 254.4 mm, vias 1 -> 3
- net Net-(U2B-B16): track 0.00 -> 44.9 mm
- net Z16: track 202.2 -> 246.3 mm
- net S3: track 196.1 -> 153.7 mm, vias 0 -> 2
- net Net-(U2B-B17): track 0.00 -> 41.8 mm
- net ~{HALT}: track 220.5 -> 179.2 mm, vias 0 -> 2
- net Net-(U2A-T2): track 0.00 -> 40.9 mm
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