File: power.kicad_sch (KiCad schematic)
At the start: 11 parts, among them J1 PWR_SWITCH, J2 PWR_LED, U1 TSN 1-2450

Commit message: board layout
Parts:
- C1: footprint Capacitor_SMD:CP_Elec_6.3x5.4_Nichicon -> Capacitor_THT:CP_Radial_D8.0mm_P5.00mm
- R1, R2: footprint Resistor_SMD:R_0805_2012Metric_Pad1.20x1.40mm_HandSolder -> Resistor_THT:R_Axial_DIN0204_L3.6mm_D1.6mm_P2.54mm_Vertical
Connections:
- net +3V3 renamed +3.3V
Changed lines of the file:
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@@
 	)
 	(symbol
-		(lib_id "power:+3V3")
+		(lib_id "power:+3.3V")
 		(at 165.1 90.17 270)
 		(unit 1)
@@
 			)
 		)
-		(property "Value" "+3V3"
+		(property "Value" "+3.3V"
 			(at 168.91 90.1699 90)
 			(effects
@@
 			)
 		)
-		(property "Description" ""
+		(property "Description" "Power symbol creates a global label with name \"+3.3V\""
 			(at 165.1 90.17 0)
 			(effects
@@
 			)
 		)
-		(property "Footprint" "Resistor_SMD:R_0805_2012Metric_Pad1.20x1.40mm_HandSolder"
+		(property "Footprint" "Resistor_THT:R_Axial_DIN0204_L3.6mm_D1.6mm_P2.54mm_Vertical"
 			(at 175.26 77.47 0)
 			(effects
@@
 			)
 		)
-		(property "Footprint" "Resistor_SMD:R_0805_2012Metric_Pad1.20x1.40mm_HandSolder"
+		(property "Footprint" "Resistor_THT:R_Axial_DIN0204_L3.6mm_D1.6mm_P2.54mm_Vertical"
 			(at 102.87 77.47 0)
 			(effects
@@
 			)
 		)
-		(property "Footprint" "Capacitor_SMD:CP_Elec_6.3x5.4_Nichicon"
+		(property "Footprint" "Capacitor_THT:CP_Radial_D8.0mm_P5.00mm"
 			(at 170.18 118.11 0)
 			(effects

Commit message: revise bus tracing
Parts:
- added C22: 10nF, Capacitor_THT:C_Disc_D3.0mm_W1.6mm_P2.50mm, symbol Device:C_Small
- added U9: 74LS112, Package_SO:SOIC-16_3.9x9.9mm_P1.27mm, symbol 74xx:74LS112
- F1, F4: DigiKey (none) -> 235-1243-ND
- F2, F3: DigiKey (none) -> RUSBF075-APHFCT-ND
- PL5: footprint Connector_Molex:Molex_Mini-Fit_Jr_5566-20A_2x10_P4.20mm_Vertical -> Connector_Molex:Molex_Mini-Fit_Jr_5566-20A2_2x10_P4.20mm_Vertical
- R1: value 4K7 -> 10K; DigiKey 541-4131-1-ND -> (none)
Connections:
- net GND: now also U9.8 (GND); no longer R1.1
- net at J1.1 (Pin_1), R1.2: now also C22.1
- net -12V: now reaches F4.2, U1.2 (VI)
- net at J1.2 (Pin_2): now also C22.2, U9.1 (C); no longer PL5.14 (PS_ON#)
- net +5VD: now reaches PL5.9 (+5VSB)
- net +5VD: now also R1.1, U9.10 (~{S}), U9.11 (J), U9.12 (K), U9.13 (C), U9.14 (~{R}), U9.15 (~{R}), U9.16 (VCC), U9.2 (K), U9.3 (J), U9.4 (~{S})
- new net: PL5.14 (PS_ON#), U9.6 (~{Q})
- no-connect marks 2 -> 4
Other:
- moved on the sheet: J1, J2
